Commit message: ok

File: spot_micro_rviz/urdf/test2.urdf (robot description, URDF)
Before this commit: robot spot_micro_rviz, 24 links, 23 joints
Links:
- link front_left_foot_link: geometry collision box size=0.026 0.020 0.13
- link front_left_leg_link: geometry collision box size=0.028 0.036 0.1075
- link front_left_leg_link_cover: geometry 
- link front_left_shoulder_link: geometry collision box size=0.044 0.038 0.07
- link front_right_foot_link: geometry collision box size=0.026 0.020 0.13
- link front_right_leg_link: geometry collision box size=0.028 0.036 0.1075
- link front_right_leg_link_cover: geometry 
- link front_right_shoulder_link: geometry collision box size=0.044 0.038 0.07
- link rear_left_foot_link: geometry collision box size=0.026 0.020 0.13
- link rear_left_leg_link: geometry collision box size=0.028 0.036 0.1075
- link rear_left_leg_link_cover: geometry 
- link rear_left_shoulder_link: geometry collision box size=0.044 0.038 0.07
- link rear_right_foot_link: geometry collision box size=0.026 0.020 0.13
- link rear_right_leg_link: geometry collision box size=0.028 0.036 0.1075
- link rear_right_leg_link_cover: geometry 
- link rear_right_shoulder_link: geometry collision box size=0.044 0.038 0.07
